Commit message: init

File: ur_description/urdf/inc/ur_macro.xacro (robot description, xacro)
@@ -136,7 +136,7 @@
       </visual>
       <collision>
-        <origin xyz="0 0 ${elbow_offset}" rpy="${pi/2} 0 ${-pi/2}"/>
-        <geometry>
-          <mesh filename="${forearm_collision_mesh}"/>
+        <origin xyz="-0.18 0 ${elbow_offset}" rpy="${pi/2} 0 ${-pi/2}"/>
+        <geometry>
+          <cylinder length="0.5" radius="0.085"/>
         </geometry>
       </collision>
@@ -308,12 +308,120 @@
       <origin xyz="0 0 0" rpy="0 ${-pi/2.0} ${-pi/2.0}" />
     </joint>
-    <!-- ROS-Industrial 'tool0' frame: all-zeros tool frame -->
-    <link name="${prefix}tool0"/>
+    <!-- Start: This setup are meant for 'air-brush' experiments -->
+    <link name="${prefix}tool0">
+      <visual>
+        <origin xyz="-0.02 -0.05 -0.115" rpy="0 0 0" />
+        <geometry>
+          <box size="0.17 0.18 0.23" />
+        </geometry>
+        <material name="green">
+          <color rgba="0 1 0 1" />
+        </material>
+      </visual>
+      <collision>
+        <origin xyz="-0.02 -0.05 -0.115" rpy="0 0 0" />
+        <geometry>
+          <box size="0.17 0.18 0.23" />
+        </geometry>
+      </collision>
+    </link>
     <joint name="${prefix}flange-tool0" type="fixed">
-      <!-- default toolframe: X+ left, Y+ up, Z+ front -->
-      <origin xyz="0 0 0" rpy="${pi/2.0} 0 ${pi/2.0}"/>
+      <origin xyz="0.23 0 -0.095" rpy="-${pi/2.0} 0 -${pi/2.0}"/>
       <parent link="${prefix}flange"/>
       <child link="${prefix}tool0"/>
     </joint>
+    <!-- End: This setup meant for 'air-brush' experiments -->
+    <!-- Start: This setup meant for 'lazer' experiments -->
+    <!-- <link name="${prefix}tool0">
+      <visual>
+        <origin xyz="-0.025 -0.04 -0.086" rpy="0 0 0" />
+        <geometry>
+          <box size="0.13 0.16 0.172" />
+        </geometry>
+        <material name="green">
+          <color rgba="0 1 0 1" />
+        </material>
+      </visual>
+      <collision>
+        <origin xyz="-0.025 -0.04 -0.086" rpy="0 0 0" />
+        <geometry>
+          <box size="0.13 0.16 0.172" />
+        </geometry>
+      </collision>
+    </link>
+    <joint name="${prefix}flange-tool0" type="fixed">
+      <origin xyz="0.172 0 -0.055" rpy="-${pi/2.0} 0 -${pi/2.0}"/>
+      <parent link="${prefix}flange"/>
+      <child link="${prefix}tool0"/>
+    </joint> -->
+    <!-- End: This setup meant for 'lazer' experiments -->
+    <!-- Start: This setup meant for 'aruco' experiments -->
+    <!-- <link name="${prefix}tool0">
+      <visual>
+        <origin xyz="0 0 -0.015" rpy="0 0 0" />
+        <geometry>
+          <box size="0.2 0.2 0.03" />
+        </geometry>
+        <material name="green">
+          <color rgba="0 1 0 1" />
+        </material>
+      </visual>
+      <collision>
+        <origin xyz="0 0 -0.015" rpy="0 0 0" />
+        <geometry>
+          <box size="0.2 0.2 0.03" />
+        </geometry>
+      </collision>
+    </link>
+    <joint name="${prefix}flange-tool0" type="fixed">
+      <origin xyz="0.014 0 0" rpy="${pi/2.0} 0 ${pi/2.0}"/>
+      <parent link="${prefix}flange"/>
+      <child link="${prefix}tool0"/>
+    </joint> -->
+    <!-- End: This setup meant for 'aruco' experiments -->
+    <link name="${prefix}table">
+      <visual>
+        <origin xyz="0 0 0.4" rpy="0 0 0" />
+        <geometry>
+          <box size="0.14 0.5 0.8" />
+        </geometry>
+        <material name="white">
+          <color rgba="1 1 1 1" />
+        </material>
+      </visual>
+      <collision>
+        <origin xyz="0 0 0.4" rpy="0 0 0" />
+        <geometry>
+         <box size="0.14 0.5 0.8" />
+        </geometry>
+      </collision>
+    </link>
+    <joint name="${prefix}table-base_link" type="fixed">
+      <origin xyz="0 0 0.8" rpy="0 0 0"/>
+      <parent link="${prefix}table"/>
+      <child link="${prefix}base_link"/>
+    </joint>
+    <link name="${prefix}camera_stand">
+      <visual>
+        <origin xyz="0 -0.16 0.045" rpy="0 0 0" />
+        <geometry>
+          <box size="0.25 0.16 0.09" />
+        </geometry>
+        <material name="blue">
+          <color rgba="0 0 1 1" />
+        </material>
+      </visual>
+      <collision>
+        <origin xyz="0 -0.16 0.045" rpy="0 0 0" />
+        <geometry>
+         <box size="0.25 0.16 0.09" />
+        </geometry>
+      </collision>
+    </link>
+    <joint name="${prefix}base_link-camera_stand" type="fixed">
+      <origin xyz="0 0 0" rpy="0 0 0"/>
+      <parent link="${prefix}base_link"/>
+      <child link="${prefix}camera_stand"/>
+    </joint>
   </xacro:macro>
 </robot>

File: ur_gazebo/urdf/ur.xacro (robot description, xacro)
@@ -64,5 +64,5 @@
   <joint name="world_joint" type="fixed">
     <parent link="world"/>
-    <child link="base_link"/>
+    <child link="table"/>
     <origin xyz="0 0 0" rpy="0 0 0"/>
   </joint>

Commit message: adding D415 camera to the scene in Rviz

File: ur_description/urdf/inc/ur_macro.xacro (robot description, xacro)
@@ -404,7 +404,7 @@
     <link name="${prefix}camera_stand">
       <visual>
-        <origin xyz="0 -0.16 0.045" rpy="0 0 0" />
-        <geometry>
-          <box size="0.25 0.16 0.09" />
+        <origin xyz="0 -0.22 0.045" rpy="${(pi/2.0)*0.75} 0 0" />
+        <geometry>
+          <mesh filename="package://realsense2_description/meshes/d415.stl"/>
         </geometry>
         <material name="blue">

Commit message: .

File: ur_description/urdf/inc/ur_macro.xacro (robot description, xacro)
@@ -311,10 +311,10 @@
     <link name="${prefix}tool0">
       <visual>
-        <origin xyz="-0.02 -0.05 -0.115" rpy="0 0 0" />
-        <geometry>
-          <box size="0.17 0.18 0.23" />
-        </geometry>
-        <material name="green">
-          <color rgba="0 1 0 1" />
+        <origin xyz="0 -0.095 -0.23" rpy="0 0 0" />
+        <geometry>
+          <mesh filename="package://gemmapp_ros/config/end_effector.stl"/>
+        </geometry>
+        <material name="air_brush_color">
+          <color rgba="1 ${186.0/255.0} ${172.0/255.0} 1" />
         </material>
       </visual>

Commit message: .

File: ur_description/urdf/inc/ur_macro.xacro (robot description, xacro)
@@ -311,5 +311,5 @@
     <link name="${prefix}tool0">
       <visual>
-        <origin xyz="0 -0.095 -0.23" rpy="0 0 0" />
+        <origin xyz="0 -0.055 -0.165" rpy="0 0 0" />
         <geometry>
           <mesh filename="package://gemmapp_ros/config/end_effector.stl"/>
@@ -320,12 +320,12 @@
       </visual>
       <collision>
-        <origin xyz="-0.02 -0.05 -0.115" rpy="0 0 0" />
-        <geometry>
-          <box size="0.17 0.18 0.23" />
+        <origin xyz="-0.02 -0.03 -0.0825" rpy="0 0 0" />
+        <geometry>
+          <box size="0.12 0.14 0.165" />
         </geometry>
       </collision>
     </link>
     <joint name="${prefix}flange-tool0" type="fixed">
-      <origin xyz="0.23 0 -0.095" rpy="-${pi/2.0} 0 -${pi/2.0}"/>
+      <origin xyz="0.165 0 -0.055" rpy="-${pi/2.0} 0 -${pi/2.0}"/>
       <parent link="${prefix}flange"/>
       <child link="${prefix}tool0"/>

Commit message: .

File: ur_description/urdf/inc/ur_macro.xacro (robot description, xacro)
@@ -311,5 +311,5 @@
     <link name="${prefix}tool0">
       <visual>
-        <origin xyz="0 -0.055 -0.165" rpy="0 0 0" />
+        <origin xyz="0 -0.059 -0.1652" rpy="0 0 0" />
         <geometry>
           <mesh filename="package://gemmapp_ros/config/end_effector.stl"/>
@@ -322,10 +322,10 @@
         <origin xyz="-0.02 -0.03 -0.0825" rpy="0 0 0" />
         <geometry>
-          <box size="0.12 0.14 0.165" />
+          <box size="0.12 0.14 0.1652" />
         </geometry>
       </collision>
     </link>
     <joint name="${prefix}flange-tool0" type="fixed">
-      <origin xyz="0.165 0 -0.055" rpy="-${pi/2.0} 0 -${pi/2.0}"/>
+      <origin xyz="0.1652 0 -0.059" rpy="-${pi/2.0} 0 -${pi/2.0}"/>
       <parent link="${prefix}flange"/>
       <child link="${prefix}tool0"/>

Commit message: .

File: ur_description/urdf/inc/ur_macro.xacro (robot description, xacro)
@@ -311,5 +311,5 @@
     <link name="${prefix}tool0">
       <visual>
-        <origin xyz="0 -0.059 -0.1652" rpy="0 0 0" />
+        <origin xyz="0 -0.059 -0.1033" rpy="0 0 0" />
         <geometry>
           <mesh filename="package://gemmapp_ros/config/end_effector.stl"/>
@@ -320,12 +320,12 @@
       </visual>
       <collision>
-        <origin xyz="-0.02 -0.03 -0.0825" rpy="0 0 0" />
-        <geometry>
-          <box size="0.12 0.14 0.1652" />
+        <origin xyz="-0.02 -0.03 -0.076" rpy="0 0 0" />
+        <geometry>
+          <box size="0.12 0.14 0.14" />
         </geometry>
       </collision>
     </link>
     <joint name="${prefix}flange-tool0" type="fixed">
-      <origin xyz="0.1652 0 -0.059" rpy="-${pi/2.0} 0 -${pi/2.0}"/>
+      <origin xyz="0.1033 0 -0.059" rpy="-${pi/2.0} 0 -${pi/2.0}"/>
       <parent link="${prefix}flange"/>
       <child link="${prefix}tool0"/>

Commit message: .

File: ur_description/urdf/inc/ur_macro.xacro (robot description, xacro)
@@ -308,8 +308,7 @@
       <origin xyz="0 0 0" rpy="0 ${-pi/2.0} ${-pi/2.0}" />
     </joint>
-    <!-- Start: This setup are meant for 'air-brush' experiments -->
-    <link name="${prefix}tool0">
-      <visual>
-        <origin xyz="0 -0.059 -0.1033" rpy="0 0 0" />
+    <link name="${prefix}tool_temp">
+      <visual>
+        <origin xyz="0 0 0" rpy="0 0 0" />
         <geometry>
           <mesh filename="package://gemmapp_ros/config/end_effector.stl"/>
@@ -320,5 +319,5 @@
       </visual>
       <collision>
-        <origin xyz="-0.02 -0.03 -0.076" rpy="0 0 0" />
+        <origin xyz="-0.02 0.03 0.025" rpy="0 0 0" />
         <geometry>
           <box size="0.12 0.14 0.14" />
@@ -326,7 +325,18 @@
       </collision>
     </link>
-    <joint name="${prefix}flange-tool0" type="fixed">
-      <origin xyz="0.1033 0 -0.059" rpy="-${pi/2.0} 0 -${pi/2.0}"/>
+    <joint name="${prefix}flange-tool_temp" type="fixed">
+      <origin xyz="0 0 0" rpy="-${pi/2.0} 0 -${pi/2.0}"/>
       <parent link="${prefix}flange"/>
+      <child link="${prefix}tool_temp"/>
+    </joint>
+    <xacro:property name="x_angle" value="0.0499584"/>
+    <xacro:property name="y_angle" value="0"/>
+    <xacro:property name="y_shift" value="0.059"/>
+    <xacro:property name="z_shift" value="0.1033"/>
+    <!-- Start: This setup are meant for 'air-brush' experiments -->
+    <link name="${prefix}tool0" />
+    <joint name="${prefix}tool_temp-tool0" type="fixed">
+      <origin xyz="0 ${y_shift} ${z_shift}" rpy="${y_angle} ${x_angle} 0"/>
+      <parent link="${prefix}tool_temp"/>
       <child link="${prefix}tool0"/>
     </joint>

Commit message: adding table the the scene

File: ur_description/urdf/inc/ur_macro.xacro (robot description, xacro)
@@ -390,23 +390,24 @@
     </joint> -->
     <!-- End: This setup meant for 'aruco' experiments -->
+    <xacro:property name="table_height" value="0.8"/>
     <link name="${prefix}table">
       <visual>
-        <origin xyz="0 0 0.4" rpy="0 0 0" />
-        <geometry>
-          <box size="0.14 0.5 0.8" />
-        </geometry>
-        <material name="white">
-          <color rgba="1 1 1 1" />
-        </material>
-      </visual>
-      <collision>
-        <origin xyz="0 0 0.4" rpy="0 0 0" />
-        <geometry>
-         <box size="0.14 0.5 0.8" />
+        <origin xyz="0 0 ${table_height}" rpy="0 0 0" />
+        <geometry>
+          <mesh filename="package://gemmapp_ros/config/round_table.stl"/>
+        </geometry>
+        <material name="table_color">
+          <color rgba="1 ${186.0/255.0} ${172.0/255.0} 1" />
+        </material>
+      </visual>
+      <collision>
+        <origin xyz="0 0 ${table_height / 2.0}" rpy="0 0 0" />
+        <geometry>
+         <box size="0.14 0.5 ${table_height}" />
         </geometry>
       </collision>
     </link>
     <joint name="${prefix}table-base_link" type="fixed">
-      <origin xyz="0 0 0.8" rpy="0 0 0"/>
+      <origin xyz="0 0 ${table_height}" rpy="0 0 0"/>
       <parent link="${prefix}table"/>
       <child link="${prefix}base_link"/>
@@ -414,7 +415,7 @@
     <link name="${prefix}camera_stand">
       <visual>
-        <origin xyz="0 -0.22 0.045" rpy="${(pi/2.0)*0.75} 0 0" />
-        <geometry>
-          <mesh filename="package://realsense2_description/meshes/d415.stl"/>
+        <origin xyz="0 -0.22 0.045" rpy="0 0 0" />
+        <geometry>
+          <mesh filename="package://gemmapp_ros/config/static_camera_D415.stl"/>
         </geometry>
         <material name="blue">

Commit message: .

File: ur_description/urdf/inc/ur_macro.xacro (robot description, xacro)
@@ -312,5 +312,5 @@
         <origin xyz="0 0 0" rpy="0 0 0" />
         <geometry>
-          <mesh filename="package://gemmapp_ros/config/end_effector.stl"/>
+          <mesh filename="package://gemmapp_ros/meshes/end_effector.stl"/>
         </geometry>
         <material name="air_brush_color">
@@ -395,5 +395,5 @@
         <origin xyz="0 0 ${table_height}" rpy="0 0 0" />
         <geometry>
-          <mesh filename="package://gemmapp_ros/config/round_table.stl"/>
+          <mesh filename="package://gemmapp_ros/meshes/round_table.stl"/>
         </geometry>
         <material name="table_color">
@@ -417,5 +417,5 @@
         <origin xyz="0 -0.22 0.045" rpy="0 0 0" />
         <geometry>
-          <mesh filename="package://gemmapp_ros/config/static_camera_D415.stl"/>
+          <mesh filename="package://gemmapp_ros/meshes/static_camera_D415.stl"/>
         </geometry>
         <material name="blue">

Commit message: adding eclipse airbrush

File: ur_description/urdf/inc/ur_macro.xacro (robot description, xacro)
@@ -312,14 +312,41 @@
         <origin xyz="0 0 0" rpy="0 0 0" />
         <geometry>
-          <mesh filename="package://gemmapp_ros/meshes/end_effector.stl"/>
-        </geometry>
-        <material name="air_brush_color">
+          <mesh filename="package://gemmapp_ros/meshes/eclipse_endeffector_airbrush.stl"/>
+        </geometry>
+        <material name="eclipse_endeffector_airbrush">
           <color rgba="1 ${186.0/255.0} ${172.0/255.0} 1" />
         </material>
       </visual>
-      <collision>
-        <origin xyz="-0.02 0.03 0.025" rpy="0 0 0" />
-        <geometry>
-          <box size="0.12 0.14 0.14" />
+      <visual>
+        <origin xyz="0 0 0" rpy="0 0 0" />
+        <geometry>
+          <mesh filename="package://gemmapp_ros/meshes/eclipse_endeffector_camera.stl"/>
+        </geometry>
+        <material name="eclipse_endeffector_camera">
+          <color rgba="${20.0/255.0} ${20.0/255.0} ${240.0/255.0} 1" />
+        </material>
+      </visual>
+      <visual>
+        <origin xyz="0 0 0" rpy="0 0 0" />
+        <geometry>
+          <mesh filename="package://gemmapp_ros/meshes/eclipse_endeffector_gripper.stl"/>
+        </geometry>
+        <material name="eclipse_endeffector_gripper">
+          <color rgba="${100.0/255.0} ${100.0/255.0} ${100.0/255.0} 1" />
+        </material>
+      </visual>
+      <visual>
+        <origin xyz="0 0 0" rpy="0 0 0" />
+        <geometry>
+          <mesh filename="package://gemmapp_ros/meshes/eclipse_endeffector_servo.stl"/>
+        </geometry>
+        <material name="eclipse_endeffector_servo">
+          <color rgba="${240.0/255.0} ${20.0/255.0} ${20.0/255.0} 1" />
+        </material>
+      </visual>
+      <collision>
+        <origin xyz="0 0 0" rpy="0 0 0" />
+        <geometry>
+          <mesh filename="package://gemmapp_ros/meshes/eclipse_endeffector_collision.stl"/>
         </geometry>
       </collision>
@@ -330,6 +357,7 @@
       <child link="${prefix}tool_temp"/>
     </joint>
-    <xacro:property name="x_angle" value="0.0499584"/>
-    <xacro:property name="y_angle" value="0"/>
+    <xacro:property name="calibration_x_angle" value="0.0499584"/>
+    <xacro:property name="calibration_y_angle" value="0"/>
+    <xacro:property name="x_shift" value="0.0"/>
     <xacro:property name="y_shift" value="0.059"/>
     <xacro:property name="z_shift" value="0.1033"/>
@@ -337,5 +365,5 @@
     <link name="${prefix}tool0" />
     <joint name="${prefix}tool_temp-tool0" type="fixed">
-      <origin xyz="0 ${y_shift} ${z_shift}" rpy="${y_angle} ${x_angle} 0"/>
+      <origin xyz="${x_shift} ${y_shift} ${z_shift}" rpy="${calibration_y_angle} ${calibration_x_angle} 0"/>
       <parent link="${prefix}tool_temp"/>
       <child link="${prefix}tool0"/>

Commit message: .

File: ur_description/urdf/inc/ur_macro.xacro (robot description, xacro)
@@ -357,9 +357,9 @@
       <child link="${prefix}tool_temp"/>
     </joint>
-    <xacro:property name="calibration_x_angle" value="0.0499584"/>
+    <xacro:property name="calibration_x_angle" value="0"/>
     <xacro:property name="calibration_y_angle" value="0"/>
     <xacro:property name="x_shift" value="0.0"/>
-    <xacro:property name="y_shift" value="0.059"/>
-    <xacro:property name="z_shift" value="0.1033"/>
+    <xacro:property name="y_shift" value="0.078"/>
+    <xacro:property name="z_shift" value="0.1224"/>
     <!-- Start: This setup are meant for 'air-brush' experiments -->
     <link name="${prefix}tool0" />

Commit message: .

File: ur_description/urdf/inc/ur_macro.xacro (robot description, xacro)
@@ -138,5 +138,11 @@
         <origin xyz="-0.18 0 ${elbow_offset}" rpy="${pi/2} 0 ${-pi/2}"/>
         <geometry>
-          <cylinder length="0.5" radius="0.085"/>
+          <cylinder length="0.35" radius="0.085"/>
+        </geometry>
+      </collision>
+       <collision>
+        <origin xyz="-0.18 0 ${elbow_offset}" rpy="${pi/2} 0 ${-pi/2}"/>
+        <geometry>
+          <cylinder length="0.5" radius="0.05"/>
         </geometry>
       </collision>
@@ -419,5 +425,56 @@
     <!-- End: This setup meant for 'aruco' experiments -->
     <xacro:property name="table_height" value="0.8"/>
+    <xacro:property name="cms_angle_degrees" value="35"/>
+    <xacro:property name="cms_angle_rad" value="${cms_angle_degrees * pi / 180.0}"/>
+    <xacro:property name="cms_angle_rad_flip" value="${pi - cms_angle_rad}"/>
+    <xacro:property name="cms_radius" value="${0.85 + 0.5}"/>
+    <xacro:property name="cms_x" value="${-cms_radius * sin(cms_angle_rad)}"/>
+    <xacro:property name="cms_y" value="${-cms_radius * cos(cms_angle_rad)}"/>
     <link name="${prefix}table">
+      <visual>
+        <origin xyz="${cms_x} ${cms_y} 0" rpy="0 0 ${cms_angle_rad_flip}" />
+        <geometry>
+          <mesh filename="package://gemmapp_ros/meshes/cms/arm.stl"/>
+        </geometry>
+        <material name="cms_arm">
+          <color rgba="${200.0/255.0} ${200.0/255.0} ${200.0/255.0} 1" />
+        </material>
+      </visual>
+      <visual>
+        <origin xyz="${cms_x} ${cms_y} 0" rpy="0 0 ${cms_angle_rad_flip}" />
+        <geometry>
+          <mesh filename="package://gemmapp_ros/meshes/cms/base.stl"/>
+        </geometry>
+        <material name="cms_base">
+          <color rgba="${100/255.0} ${100/255.0} ${100/255.0} 1" />
+        </material>
+      </visual>
+      <visual>
+        <origin xyz="${cms_x} ${cms_y} 0" rpy="0 0 ${cms_angle_rad_flip}" />
+        <geometry>
+          <mesh filename="package://gemmapp_ros/meshes/cms/cms1.stl"/>
+        </geometry>
+        <material name="cms_cms1">
+          <color rgba="${100/255.0} ${100/255.0} ${100/255.0} 1" />
+        </material>
+      </visual>
+      <visual>
+        <origin xyz="${cms_x} ${cms_y} 0" rpy="0 0 ${cms_angle_rad_flip}" />
+        <geometry>
+          <mesh filename="package://gemmapp_ros/meshes/cms/cms2.stl"/>
+        </geometry>
+        <material name="cms_cms2">
+          <color rgba="${200.0/255.0} ${200.0/255.0} ${200.0/255.0} 1" />
+        </material>
+      </visual>
+      <visual>
+        <origin xyz="${cms_x} ${cms_y} 0" rpy="0 0 ${cms_angle_rad_flip}" />
+        <geometry>
+          <mesh filename="package://gemmapp_ros/meshes/cms/cms3.stl"/>
+        </geometry>
+        <material name="cms_cms3">
+          <color rgba="${100/255.0} ${100/255.0} ${100/255.0} 1" />
+        </material>
+      </visual>
       <visual>
         <origin xyz="0 0 ${table_height}" rpy="0 0 0" />

Commit message: .

File: ur_description/urdf/inc/ur_macro.xacro (robot description, xacro)
@@ -376,28 +376,4 @@
     </joint>
     <!-- End: This setup meant for 'air-brush' experiments -->
-    <!-- Start: This setup meant for 'lazer' experiments -->
-    <!-- <link name="${prefix}tool0">
-      <visual>
-        <origin xyz="-0.025 -0.04 -0.086" rpy="0 0 0" />
-        <geometry>
-          <box size="0.13 0.16 0.172" />
-        </geometry>
-        <material name="green">
-          <color rgba="0 1 0 1" />
-        </material>
-      </visual>
-      <collision>
-        <origin xyz="-0.025 -0.04 -0.086" rpy="0 0 0" />
-        <geometry>
-          <box size="0.13 0.16 0.172" />
-        </geometry>
-      </collision>
-    </link>
-    <joint name="${prefix}flange-tool0" type="fixed">
-      <origin xyz="0.172 0 -0.055" rpy="-${pi/2.0} 0 -${pi/2.0}"/>
-      <parent link="${prefix}flange"/>
-      <child link="${prefix}tool0"/>
-    </joint> -->
-    <!-- End: This setup meant for 'lazer' experiments -->
     <!-- Start: This setup meant for 'aruco' experiments -->
     <!-- <link name="${prefix}tool0">
@@ -500,5 +476,5 @@
     <link name="${prefix}camera_stand">
       <visual>
-        <origin xyz="0 -0.22 0.045" rpy="0 0 0" />
+        <origin xyz="0 0 0" rpy="0 0 0" />
         <geometry>
           <mesh filename="package://gemmapp_ros/meshes/static_camera_D415.stl"/>
@@ -509,12 +485,12 @@
       </visual>
       <collision>
-        <origin xyz="0 -0.16 0.045" rpy="0 0 0" />
-        <geometry>
-         <box size="0.25 0.16 0.09" />
+        <origin xyz="-0.02 0 0" rpy="0 0 0" />
+        <geometry>
+         <box size="0.12 0.04 0.04" />
         </geometry>
       </collision>
     </link>
     <joint name="${prefix}base_link-camera_stand" type="fixed">
-      <origin xyz="0 0 0" rpy="0 0 0"/>
+      <origin xyz="0.03714007037884025 -0.11853391014676645 0.06885225109582538" rpy="0 0 0"/>
       <parent link="${prefix}base_link"/>
       <child link="${prefix}camera_stand"/>
