Commit message: .

File: ur_description/urdf/inc/ur_macro.xacro (robot description, xacro)
@@ -401,13 +401,12 @@
     <!-- End: This setup meant for 'aruco' experiments -->
     <xacro:property name="table_height" value="0.8"/>
-    <xacro:property name="cms_angle_degrees" value="35"/>
-    <xacro:property name="cms_angle_rad" value="${cms_angle_degrees * pi / 180.0}"/>
-    <xacro:property name="cms_angle_rad_flip" value="${pi - cms_angle_rad}"/>
-    <xacro:property name="cms_radius" value="${0.85 + 0.5}"/>
-    <xacro:property name="cms_x" value="${-cms_radius * sin(cms_angle_rad)}"/>
-    <xacro:property name="cms_y" value="${-cms_radius * cos(cms_angle_rad)}"/>
+    <xacro:property name="cms_angle_degrees" value="50"/>
+    <xacro:property name="cms_flipped_angle_rad" value="${(180.0 - cms_angle_degrees) * pi / 180.0}"/>
+    <xacro:property name="cms_x" value="-0.712"/>
+    <xacro:property name="cms_y" value="-0.598"/>
+    <xacro:property name="cms_z" value="${0.275 + table_height}"/>
     <link name="${prefix}table">
       <visual>
-        <origin xyz="${cms_x} ${cms_y} 0" rpy="0 0 ${cms_angle_rad_flip}" />
+        <origin xyz="${cms_x} ${cms_y} ${cms_z}" rpy="0 0 ${cms_flipped_angle_rad}" />
         <geometry>
           <mesh filename="package://gemmapp_ros/meshes/cms/arm.stl"/>
@@ -418,5 +417,5 @@
       </visual>
       <visual>
-        <origin xyz="${cms_x} ${cms_y} 0" rpy="0 0 ${cms_angle_rad_flip}" />
+        <origin xyz="${cms_x} ${cms_y} ${cms_z}" rpy="0 0 ${cms_flipped_angle_rad}" />
         <geometry>
           <mesh filename="package://gemmapp_ros/meshes/cms/base.stl"/>
@@ -427,5 +426,5 @@
       </visual>
       <visual>
-        <origin xyz="${cms_x} ${cms_y} 0" rpy="0 0 ${cms_angle_rad_flip}" />
+        <origin xyz="${cms_x} ${cms_y} ${cms_z}" rpy="0 0 ${cms_flipped_angle_rad}" />
         <geometry>
           <mesh filename="package://gemmapp_ros/meshes/cms/cms1.stl"/>
@@ -436,5 +435,5 @@
       </visual>
       <visual>
-        <origin xyz="${cms_x} ${cms_y} 0" rpy="0 0 ${cms_angle_rad_flip}" />
+        <origin xyz="${cms_x} ${cms_y} ${cms_z}" rpy="0 0 ${cms_flipped_angle_rad}" />
         <geometry>
           <mesh filename="package://gemmapp_ros/meshes/cms/cms2.stl"/>
@@ -445,5 +444,5 @@
       </visual>
       <visual>
-        <origin xyz="${cms_x} ${cms_y} 0" rpy="0 0 ${cms_angle_rad_flip}" />
+        <origin xyz="${cms_x} ${cms_y} ${cms_z}" rpy="0 0 ${cms_flipped_angle_rad}" />
         <geometry>
           <mesh filename="package://gemmapp_ros/meshes/cms/cms3.stl"/>
@@ -453,4 +452,22 @@
         </material>
       </visual>
+      <collision>
+        <origin xyz="${cms_x} ${cms_y} ${cms_z}" rpy="0 0 ${cms_flipped_angle_rad}" />
+        <geometry>
+          <mesh filename="package://gemmapp_ros/meshes/cms/collision_up.stl"/>
+        </geometry>
+      </collision>
+      <collision>
+        <origin xyz="${cms_x} ${cms_y} ${cms_z}" rpy="0 0 ${cms_flipped_angle_rad}" />
+        <geometry>
+          <mesh filename="package://gemmapp_ros/meshes/cms/collision_down.stl"/>
+        </geometry>
+      </collision>
+      <collision>
+        <origin xyz="${cms_x} ${cms_y} ${cms_z}" rpy="0 0 ${cms_flipped_angle_rad}" />
+        <geometry>
+          <mesh filename="package://gemmapp_ros/meshes/cms/arm.stl"/>
+        </geometry>
+      </collision>
       <visual>
         <origin xyz="0 0 ${table_height}" rpy="0 0 0" />
@@ -478,8 +495,17 @@
         <origin xyz="0 0 0" rpy="0 0 0" />
         <geometry>
-          <mesh filename="package://gemmapp_ros/meshes/static_camera_D415.stl"/>
-        </geometry>
-        <material name="blue">
-          <color rgba="0 0 1 1" />
+          <mesh filename="package://gemmapp_ros/meshes/static_camera/D415.stl"/>
+        </geometry>
+        <material name="static_camera_D415">
+          <color rgba="${70/255.0} ${70/255.0} ${200.0/255.0} 1" />
+        </material>
+      </visual>
+      <visual>
+        <origin xyz="0 0 0" rpy="0 0 0" />
+        <geometry>
+          <mesh filename="package://gemmapp_ros/meshes/static_camera/arm.stl"/>
+        </geometry>
+        <material name="static_camera_arm">
+          <color rgba="${80.0/255.0} ${80.0/255.0} ${80.0/255.0} 1" />
         </material>
       </visual>

Commit message: adding humn to the scene

File: ur_description/urdf/inc/ur_macro.xacro (robot description, xacro)
@@ -406,5 +406,26 @@
     <xacro:property name="cms_y" value="-0.598"/>
     <xacro:property name="cms_z" value="${0.275 + table_height}"/>
+    <xacro:property name="woman_x" value="0.0"/>
+    <xacro:property name="woman_y" value="-0.6"/>
+    <xacro:property name="woman_z" value="${0.45 + table_height}"/>
     <link name="${prefix}table">
+      <!-- <visual>
+        <origin xyz="${woman_x} ${woman_y} ${woman_z}" rpy="0 0 0" />
+        <geometry>
+          <mesh filename="package://gemmapp_ros/meshes/human/chair.stl"/>
+        </geometry>
+        <material name="cms_arm">
+          <color rgba="${200.0/255.0} ${200.0/255.0} ${200.0/255.0} 1" />
+        </material>
+      </visual>
+      <visual>
+        <origin xyz="${woman_x} ${woman_y} ${woman_z}" rpy="0 0 0" />
+        <geometry>
+          <mesh filename="package://gemmapp_ros/meshes/human/woman.stl"/>
+        </geometry>
+        <material name="cms_arm">
+          <color rgba="${200.0/255.0} ${200.0/255.0} ${200.0/255.0} 1" />
+        </material>
+      </visual> -->
       <visual>
         <origin xyz="${cms_x} ${cms_y} ${cms_z}" rpy="0 0 ${cms_flipped_angle_rad}" />

Commit message: .

File: ur_description/urdf/inc/ur_macro.xacro (robot description, xacro)
@@ -318,5 +318,5 @@
         <origin xyz="0 0 0" rpy="0 0 0" />
         <geometry>
-          <mesh filename="package://gemmapp_ros/meshes/eclipse_endeffector_airbrush.stl"/>
+          <mesh filename="package://gemmapp_ros/meshes/ee/eclipse_endeffector_airbrush.stl"/>
         </geometry>
         <material name="eclipse_endeffector_airbrush">
@@ -327,5 +327,5 @@
         <origin xyz="0 0 0" rpy="0 0 0" />
         <geometry>
-          <mesh filename="package://gemmapp_ros/meshes/eclipse_endeffector_camera.stl"/>
+          <mesh filename="package://gemmapp_ros/meshes/ee/eclipse_endeffector_camera.stl"/>
         </geometry>
         <material name="eclipse_endeffector_camera">
@@ -336,5 +336,5 @@
         <origin xyz="0 0 0" rpy="0 0 0" />
         <geometry>
-          <mesh filename="package://gemmapp_ros/meshes/eclipse_endeffector_gripper.stl"/>
+          <mesh filename="package://gemmapp_ros/meshes/ee/eclipse_endeffector_gripper.stl"/>
         </geometry>
         <material name="eclipse_endeffector_gripper">
@@ -345,5 +345,5 @@
         <origin xyz="0 0 0" rpy="0 0 0" />
         <geometry>
-          <mesh filename="package://gemmapp_ros/meshes/eclipse_endeffector_servo.stl"/>
+          <mesh filename="package://gemmapp_ros/meshes/ee/eclipse_endeffector_servo.stl"/>
         </geometry>
         <material name="eclipse_endeffector_servo">
@@ -354,5 +354,11 @@
         <origin xyz="0 0 0" rpy="0 0 0" />
         <geometry>
-          <mesh filename="package://gemmapp_ros/meshes/eclipse_endeffector_collision.stl"/>
+          <mesh filename="package://gemmapp_ros/meshes/ee/eclipse_endeffector_collision1.stl"/>
+        </geometry>
+      </collision>
+      <collision>
+        <origin xyz="0 0 0" rpy="0 0 0" />
+        <geometry>
+          <mesh filename="package://gemmapp_ros/meshes/ee/eclipse_endeffector_collision2.stl"/>
         </geometry>
       </collision>

Commit message: remove statuc camera

File: ur_description/urdf/inc/ur_macro.xacro (robot description, xacro)
@@ -518,35 +518,4 @@
       <child link="${prefix}base_link"/>
     </joint>
-    <link name="${prefix}camera_stand">
-      <visual>
-        <origin xyz="0 0 0" rpy="0 0 0" />
-        <geometry>
-          <mesh filename="package://gemmapp_ros/meshes/static_camera/D415.stl"/>
-        </geometry>
-        <material name="static_camera_D415">
-          <color rgba="${70/255.0} ${70/255.0} ${200.0/255.0} 1" />
-        </material>
-      </visual>
-      <visual>
-        <origin xyz="0 0 0" rpy="0 0 0" />
-        <geometry>
-          <mesh filename="package://gemmapp_ros/meshes/static_camera/arm.stl"/>
-        </geometry>
-        <material name="static_camera_arm">
-          <color rgba="${80.0/255.0} ${80.0/255.0} ${80.0/255.0} 1" />
-        </material>
-      </visual>
-      <collision>
-        <origin xyz="-0.02 0 0" rpy="0 0 0" />
-        <geometry>
-         <box size="0.12 0.04 0.04" />
-        </geometry>
-      </collision>
-    </link>
-    <joint name="${prefix}base_link-camera_stand" type="fixed">
-      <origin xyz="0.03714007037884025 -0.11853391014676645 0.06885225109582538" rpy="0 0 0"/>
-      <parent link="${prefix}base_link"/>
-      <child link="${prefix}camera_stand"/>
-    </joint>
   </xacro:macro>
 </robot>

Commit message: rotating table

File: ur_description/urdf/inc/ur_macro.xacro (robot description, xacro)
@@ -507,5 +507,5 @@
       </visual>
       <collision>
-        <origin xyz="0 0 ${table_height / 2.0}" rpy="0 0 0" />
+        <origin xyz="0 0 ${table_height / 2.0}" rpy="0 0 ${pi / 2.0}" />
         <geometry>
          <box size="0.14 0.5 ${table_height}" />

Commit message: adding link for camera

File: ur_description/urdf/inc/ur_macro.xacro (robot description, xacro)
@@ -369,4 +369,10 @@
       <child link="${prefix}tool_temp"/>
     </joint>
+    <link name="${prefix}camera_ee" />
+    <joint name="${prefix}tool_temp-camera_ee" type="fixed">
+      <origin xyz="0 0 0.04" rpy="0 0 0"/>
+      <parent link="${prefix}tool_temp"/>
+      <child link="${prefix}camera_ee"/>
+    </joint>
     <xacro:property name="calibration_x_angle" value="0"/>
     <xacro:property name="calibration_y_angle" value="0"/>

Commit message: adding temptu

File: ur_description/urdf/inc/ur_macro.xacro (robot description, xacro)
@@ -318,11 +318,11 @@
         <origin xyz="0 0 0" rpy="0 0 0" />
         <geometry>
-          <mesh filename="package://gemmapp_ros/meshes/ee/eclipse_endeffector_airbrush.stl"/>
-        </geometry>
-        <material name="eclipse_endeffector_airbrush">
+          <mesh filename="package://gemmapp_ros/meshes/ee/temptu_airpod_airbrush.stl"/>
+        </geometry>
+        <material name="temptu_airpod_airbrush">
           <color rgba="1 ${186.0/255.0} ${172.0/255.0} 1" />
         </material>
       </visual>
-      <visual>
+      <!-- <visual>
         <origin xyz="0 0 0" rpy="0 0 0" />
         <geometry>
@@ -332,15 +332,15 @@
           <color rgba="${20.0/255.0} ${20.0/255.0} ${240.0/255.0} 1" />
         </material>
-      </visual>
-      <visual>
-        <origin xyz="0 0 0" rpy="0 0 0" />
-        <geometry>
-          <mesh filename="package://gemmapp_ros/meshes/ee/eclipse_endeffector_gripper.stl"/>
-        </geometry>
-        <material name="eclipse_endeffector_gripper">
+      </visual> -->
+      <visual>
+        <origin xyz="0 0 0" rpy="0 0 0" />
+        <geometry>
+          <mesh filename="package://gemmapp_ros/meshes/ee/temptu_airpod_gripper.stl"/>
+        </geometry>
+        <material name="temptu_airpod_gripper">
           <color rgba="${100.0/255.0} ${100.0/255.0} ${100.0/255.0} 1" />
         </material>
       </visual>
-      <visual>
+      <!-- <visual>
         <origin xyz="0 0 0" rpy="0 0 0" />
         <geometry>
@@ -350,15 +350,15 @@
           <color rgba="${240.0/255.0} ${20.0/255.0} ${20.0/255.0} 1" />
         </material>
-      </visual>
-      <collision>
-        <origin xyz="0 0 0" rpy="0 0 0" />
-        <geometry>
-          <mesh filename="package://gemmapp_ros/meshes/ee/eclipse_endeffector_collision1.stl"/>
-        </geometry>
-      </collision>
-      <collision>
-        <origin xyz="0 0 0" rpy="0 0 0" />
-        <geometry>
-          <mesh filename="package://gemmapp_ros/meshes/ee/eclipse_endeffector_collision2.stl"/>
+      </visual> -->
+      <!-- <collision>
+        <origin xyz="0 0 0" rpy="0 0 0" />
+        <geometry>
+          <mesh filename="package://gemmapp_ros/meshes/ee/eclipse_endeffector_camera.stl"/>
+        </geometry>
+      </collision> -->
+      <collision>
+        <origin xyz="0 0 0" rpy="0 0 0" />
+        <geometry>
+          <mesh filename="package://gemmapp_ros/meshes/ee/temptu_airpod_collision.stl"/>
         </geometry>
       </collision>
@@ -378,6 +378,6 @@
     <xacro:property name="calibration_y_angle" value="0"/>
     <xacro:property name="x_shift" value="0.0"/>
-    <xacro:property name="y_shift" value="0.078"/>
-    <xacro:property name="z_shift" value="0.1224"/>
+    <xacro:property name="y_shift" value="0.0854"/>
+    <xacro:property name="z_shift" value="0.14778"/>
     <!-- Start: This setup are meant for 'air-brush' experiments -->
     <link name="${prefix}tool0" />

Commit message: adding new airpod

File: ur_description/urdf/inc/ur_macro.xacro (robot description, xacro)
@@ -324,4 +324,13 @@
         </material>
       </visual>
+      <visual>
+        <origin xyz="0 0 0" rpy="0 0 0" />
+        <geometry>
+          <mesh filename="package://gemmapp_ros/meshes/ee/temptu_airpod_camera.stl"/>
+        </geometry>
+        <material name="temptu_airpod_camera">
+          <color rgba="${20.0/255.0} ${20.0/255.0} ${240.0/255.0} 1" />
+        </material>
+      </visual>
       <!-- <visual>
         <origin xyz="0 0 0" rpy="0 0 0" />
@@ -378,5 +387,5 @@
     <xacro:property name="calibration_y_angle" value="0"/>
     <xacro:property name="x_shift" value="0.0"/>
-    <xacro:property name="y_shift" value="0.0854"/>
+    <xacro:property name="y_shift" value="0.0"/>
     <xacro:property name="z_shift" value="0.14778"/>
     <!-- Start: This setup are meant for 'air-brush' experiments -->

Commit message: moveing camera

File: ur_description/urdf/inc/ur_macro.xacro (robot description, xacro)
@@ -380,5 +380,5 @@
     <link name="${prefix}camera_ee" />
     <joint name="${prefix}tool_temp-camera_ee" type="fixed">
-      <origin xyz="0 0 0.04" rpy="0 0 0"/>
+      <origin xyz="0 -0.038 0.139" rpy="0 0 0"/>
       <parent link="${prefix}tool_temp"/>
       <child link="${prefix}camera_ee"/>

Commit message: air-brush calibration

File: ur_description/urdf/inc/ur_macro.xacro (robot description, xacro)
@@ -384,9 +384,9 @@
       <child link="${prefix}camera_ee"/>
     </joint>
-    <xacro:property name="calibration_x_angle" value="0"/>
-    <xacro:property name="calibration_y_angle" value="0"/>
+    <xacro:property name="calibration_x_angle" value="-0.0572047"/>
+    <xacro:property name="calibration_y_angle" value="-0.0290007"/>
     <xacro:property name="x_shift" value="0.0"/>
-    <xacro:property name="y_shift" value="0.0"/>
-    <xacro:property name="z_shift" value="0.14778"/>
+    <xacro:property name="y_shift" value="0.017"/>
+    <xacro:property name="z_shift" value="0.15578"/>
     <!-- Start: This setup are meant for 'air-brush' experiments -->
     <link name="${prefix}tool0" />

Commit message: add face_link

File: ur_description/urdf/inc/ur_macro.xacro (robot description, xacro)
@@ -333,13 +333,4 @@
         </material>
       </visual>
-      <!-- <visual>
-        <origin xyz="0 0 0" rpy="0 0 0" />
-        <geometry>
-          <mesh filename="package://gemmapp_ros/meshes/ee/eclipse_endeffector_camera.stl"/>
-        </geometry>
-        <material name="eclipse_endeffector_camera">
-          <color rgba="${20.0/255.0} ${20.0/255.0} ${240.0/255.0} 1" />
-        </material>
-      </visual> -->
       <visual>
         <origin xyz="0 0 0" rpy="0 0 0" />
@@ -351,19 +342,4 @@
         </material>
       </visual>
-      <!-- <visual>
-        <origin xyz="0 0 0" rpy="0 0 0" />
-        <geometry>
-          <mesh filename="package://gemmapp_ros/meshes/ee/eclipse_endeffector_servo.stl"/>
-        </geometry>
-        <material name="eclipse_endeffector_servo">
-          <color rgba="${240.0/255.0} ${20.0/255.0} ${20.0/255.0} 1" />
-        </material>
-      </visual> -->
-      <!-- <collision>
-        <origin xyz="0 0 0" rpy="0 0 0" />
-        <geometry>
-          <mesh filename="package://gemmapp_ros/meshes/ee/eclipse_endeffector_camera.stl"/>
-        </geometry>
-      </collision> -->
       <collision>
         <origin xyz="0 0 0" rpy="0 0 0" />
@@ -431,8 +407,8 @@
     <xacro:property name="woman_z" value="${0.45 + table_height}"/>
     <link name="${prefix}table">
-      <!-- <visual>
-        <origin xyz="${woman_x} ${woman_y} ${woman_z}" rpy="0 0 0" />
-        <geometry>
-          <mesh filename="package://gemmapp_ros/meshes/human/chair.stl"/>
+      <visual>
+        <origin xyz="${cms_x} ${cms_y} ${cms_z}" rpy="0 0 ${cms_flipped_angle_rad}" />
+        <geometry>
+          <mesh filename="package://gemmapp_ros/meshes/cms/arm.stl"/>
         </geometry>
         <material name="cms_arm">
@@ -441,22 +417,4 @@
       </visual>
       <visual>
-        <origin xyz="${woman_x} ${woman_y} ${woman_z}" rpy="0 0 0" />
-        <geometry>
-          <mesh filename="package://gemmapp_ros/meshes/human/woman.stl"/>
-        </geometry>
-        <material name="cms_arm">
-          <color rgba="${200.0/255.0} ${200.0/255.0} ${200.0/255.0} 1" />
-        </material>
-      </visual> -->
-      <visual>
-        <origin xyz="${cms_x} ${cms_y} ${cms_z}" rpy="0 0 ${cms_flipped_angle_rad}" />
-        <geometry>
-          <mesh filename="package://gemmapp_ros/meshes/cms/arm.stl"/>
-        </geometry>
-        <material name="cms_arm">
-          <color rgba="${200.0/255.0} ${200.0/255.0} ${200.0/255.0} 1" />
-        </material>
-      </visual>
-      <visual>
         <origin xyz="${cms_x} ${cms_y} ${cms_z}" rpy="0 0 ${cms_flipped_angle_rad}" />
         <geometry>
@@ -528,4 +486,28 @@
       </collision>
     </link>
+    <link name="face_link">
+        <visual>
+        <origin xyz="0 0 0" rpy="0 0 0" />
+        <geometry>
+          <mesh filename="file:///home/nizan/catkin_ws/src/face_scanner_ros/data/eliane_aligned_subdivision.dae"/>
+        </geometry>
+      </visual>
+      <collision>
+        <origin xyz="0 0 0" rpy="0 0 0" />
+        <geometry>
+          <mesh filename="file:///home/nizan/catkin_ws/src/face_scanner_ros/data/eliane_aligned_collision.dae"/>
+        </geometry>
+      </collision>
+      <inertial>
+            <origin rpy="0 0 0" xyz="0.043 0.001 0.002" />
+            <mass value="0.1" />
+            <inertia ixx="0.000348958333333" ixy="0" ixz="0" iyy="0.000348958333333" iyz="0" izz="3.125e-05" />
+        </inertial>
+    </link>
+    <joint name="face_joint" type="fixed">
+    <parent link="${prefix}base_link"/>
+    <child link="face_link"/>
+    <origin rpy="${pi / 2} 0 ${pi}" xyz="0 -0.55 0.45"/>
+    </joint>
     <joint name="${prefix}table-base_link" type="fixed">
       <origin xyz="0 0 ${table_height}" rpy="0 0 0"/>

Commit message: .

File: ur_description/urdf/inc/ur_macro.xacro (robot description, xacro)
@@ -490,11 +490,11 @@
         <origin xyz="0 0 0" rpy="0 0 0" />
         <geometry>
-          <mesh filename="file:///home/nizan/catkin_ws/src/face_scanner_ros/data/eliane_aligned_subdivision.dae"/>
-        </geometry>
-      </visual>
-      <collision>
-        <origin xyz="0 0 0" rpy="0 0 0" />
-        <geometry>
-          <mesh filename="file:///home/nizan/catkin_ws/src/face_scanner_ros/data/eliane_aligned_collision.dae"/>
+          <mesh filename="file:///home/nizan/catkin_ws/src/face_scanner_ros/face_database/eliane/eliane_aligned_subdivision.dae"/>
+        </geometry>
+      </visual>
+      <collision>
+        <origin xyz="0 0 0" rpy="0 0 0" />
+        <geometry>
+          <mesh filename="file:///home/nizan/catkin_ws/src/face_scanner_ros/face_database/eliane/eliane_aligned_collision.dae"/>
         </geometry>
       </collision>
