Commit message: .

File: ur_description/urdf/inc/ur_macro.xacro (robot description, xacro)
@@ -342,10 +342,10 @@
         </material>
       </visual>
-      <collision>
+      <!-- <collision>
         <origin xyz="0 0 0" rpy="0 0 0" />
         <geometry>
           <mesh filename="package://gemmapp_ros/meshes/ee/temptu_airpod_collision.stl"/>
         </geometry>
-      </collision>
+      </collision> -->
     </link>
     <joint name="${prefix}flange-tool_temp" type="fixed">
@@ -397,90 +397,19 @@
     </joint> -->
     <!-- End: This setup meant for 'aruco' experiments -->
-    <xacro:property name="table_height" value="0.8"/>
-    <xacro:property name="cms_angle_degrees" value="50"/>
-    <xacro:property name="cms_flipped_angle_rad" value="${(180.0 - cms_angle_degrees) * pi / 180.0}"/>
-    <xacro:property name="cms_x" value="-0.712"/>
-    <xacro:property name="cms_y" value="-0.598"/>
-    <xacro:property name="cms_z" value="${0.275 + table_height}"/>
-    <xacro:property name="woman_x" value="0.0"/>
-    <xacro:property name="woman_y" value="-0.6"/>
-    <xacro:property name="woman_z" value="${0.45 + table_height}"/>
+    <xacro:property name="table_height" value="0.77"/>
+    <xacro:property name="face_x" value="0"/>
+    <xacro:property name="face_y" value="-0.55"/>
+    <xacro:property name="face_z" value="0.45"/>
     <link name="${prefix}table">
       <visual>
-        <origin xyz="${cms_x} ${cms_y} ${cms_z}" rpy="0 0 ${cms_flipped_angle_rad}" />
-        <geometry>
-          <mesh filename="package://gemmapp_ros/meshes/cms/arm.stl"/>
-        </geometry>
-        <material name="cms_arm">
-          <color rgba="${200.0/255.0} ${200.0/255.0} ${200.0/255.0} 1" />
-        </material>
-      </visual>
-      <visual>
-        <origin xyz="${cms_x} ${cms_y} ${cms_z}" rpy="0 0 ${cms_flipped_angle_rad}" />
-        <geometry>
-          <mesh filename="package://gemmapp_ros/meshes/cms/base.stl"/>
-        </geometry>
-        <material name="cms_base">
-          <color rgba="${100/255.0} ${100/255.0} ${100/255.0} 1" />
-        </material>
-      </visual>
-      <visual>
-        <origin xyz="${cms_x} ${cms_y} ${cms_z}" rpy="0 0 ${cms_flipped_angle_rad}" />
-        <geometry>
-          <mesh filename="package://gemmapp_ros/meshes/cms/cms1.stl"/>
-        </geometry>
-        <material name="cms_cms1">
-          <color rgba="${100/255.0} ${100/255.0} ${100/255.0} 1" />
-        </material>
-      </visual>
-      <visual>
-        <origin xyz="${cms_x} ${cms_y} ${cms_z}" rpy="0 0 ${cms_flipped_angle_rad}" />
-        <geometry>
-          <mesh filename="package://gemmapp_ros/meshes/cms/cms2.stl"/>
-        </geometry>
-        <material name="cms_cms2">
-          <color rgba="${200.0/255.0} ${200.0/255.0} ${200.0/255.0} 1" />
-        </material>
-      </visual>
-      <visual>
-        <origin xyz="${cms_x} ${cms_y} ${cms_z}" rpy="0 0 ${cms_flipped_angle_rad}" />
-        <geometry>
-          <mesh filename="package://gemmapp_ros/meshes/cms/cms3.stl"/>
-        </geometry>
-        <material name="cms_cms3">
-          <color rgba="${100/255.0} ${100/255.0} ${100/255.0} 1" />
-        </material>
-      </visual>
-      <collision>
-        <origin xyz="${cms_x} ${cms_y} ${cms_z}" rpy="0 0 ${cms_flipped_angle_rad}" />
-        <geometry>
-          <mesh filename="package://gemmapp_ros/meshes/cms/collision_up.stl"/>
-        </geometry>
-      </collision>
-      <collision>
-        <origin xyz="${cms_x} ${cms_y} ${cms_z}" rpy="0 0 ${cms_flipped_angle_rad}" />
-        <geometry>
-          <mesh filename="package://gemmapp_ros/meshes/cms/collision_down.stl"/>
-        </geometry>
-      </collision>
-      <collision>
-        <origin xyz="${cms_x} ${cms_y} ${cms_z}" rpy="0 0 ${cms_flipped_angle_rad}" />
-        <geometry>
-          <mesh filename="package://gemmapp_ros/meshes/cms/arm.stl"/>
-        </geometry>
-      </collision>
-      <visual>
         <origin xyz="0 0 ${table_height}" rpy="0 0 0" />
         <geometry>
-          <mesh filename="package://gemmapp_ros/meshes/round_table.stl"/>
-        </geometry>
-        <material name="table_color">
-          <color rgba="${200.0/255.0} ${200.0/255.0} ${200.0/255.0} 1" />
-        </material>
-      </visual>
-      <collision>
-        <origin xyz="0 0 ${table_height / 2.0}" rpy="0 0 ${pi / 2.0}" />
-        <geometry>
-         <box size="0.14 0.5 ${table_height}" />
+          <mesh filename="file:///home/nizan/catkin_ws/src/gemmaD_robot_ros/gemmad_robot_description/stl/table/full_table.dae"/>
+        </geometry>
+      </visual>
+      <collision>
+        <origin xyz="0 0 ${table_height}" rpy="0 0 0" />
+        <geometry>
+          <mesh filename="file:///home/nizan/catkin_ws/src/gemmaD_robot_ros/gemmad_robot_description/stl/table/full_table.dae"/>
         </geometry>
       </collision>
@@ -490,5 +419,5 @@
         <origin xyz="0 0 0" rpy="0 0 0" />
         <geometry>
-          <mesh filename="file:///home/nizan/catkin_ws/src/face_scanner_ros/face_database/eliane/eliane_aligned_subdivision.dae"/>
+          <mesh filename="file:///home/nizan/catkin_ws/src/face_scanner_ros/face_database/full_body/full_body_with_chair.dae"/>
         </geometry>
       </visual>
@@ -508,5 +437,5 @@
     <parent link="${prefix}base_link"/>
     <child link="face_link"/>
-    <origin rpy="${pi / 2} 0 ${pi}" xyz="0 -0.55 0.45"/>
+    <origin rpy="${pi / 2} 0 ${pi}" xyz="${face_x} ${face_y} ${face_z}"/>
     </joint>
     <joint name="${prefix}table-base_link" type="fixed">

Commit message: limit joints & reposition face

File: ur_description/urdf/inc/ur_macro.xacro (robot description, xacro)
@@ -399,5 +399,5 @@
     <xacro:property name="table_height" value="0.77"/>
     <xacro:property name="face_x" value="0"/>
-    <xacro:property name="face_y" value="-0.55"/>
+    <xacro:property name="face_y" value="-0.70"/>
     <xacro:property name="face_z" value="0.45"/>
     <link name="${prefix}table">

Commit message: .

File: ur_description/urdf/inc/ur_macro.xacro (robot description, xacro)
@@ -342,10 +342,10 @@
         </material>
       </visual>
-      <!-- <collision>
+      <collision>
         <origin xyz="0 0 0" rpy="0 0 0" />
         <geometry>
           <mesh filename="package://gemmapp_ros/meshes/ee/temptu_airpod_collision.stl"/>
         </geometry>
-      </collision> -->
+      </collision>
     </link>
     <joint name="${prefix}flange-tool_temp" type="fixed">
@@ -415,9 +415,9 @@
       </collision>
     </link>
-    <link name="face_link">
+    <!-- <link name="face_link">
         <visual>
         <origin xyz="0 0 0" rpy="0 0 0" />
         <geometry>
-          <mesh filename="file:///home/nizan/catkin_ws/src/face_scanner_ros/face_database/full_body/full_body_with_chair.dae"/>
+          <mesh filename="file:///home/nizan/catkin_ws/src/face_scanner_ros/face_database/eliane/eliane_aligned.dae"/>
         </geometry>
       </visual>
@@ -433,10 +433,35 @@
             <inertia ixx="0.000348958333333" ixy="0" ixz="0" iyy="0.000348958333333" iyz="0" izz="3.125e-05" />
         </inertial>
-    </link>
-    <joint name="face_joint" type="fixed">
+    </link> -->
+    <!-- <link name="bust_link">
+      <collision>
+      <origin xyz="0 0 0" rpy="0 0 0" />
+      <geometry>
+          <mesh filename="file:///home/nizan/catkin_ws/src/face_scanner_ros/face_database/bust/bust_collision1.stl"/>
+      </geometry>
+      </collision>
+      <collision>
+      <origin xyz="0 0 0" rpy="0 0 0" />
+      <geometry>
+          <mesh filename="file:///home/nizan/catkin_ws/src/face_scanner_ros/face_database/bust/bust_collision2.stl"/>
+      </geometry>
+      </collision>
+      <collision>
+      <origin xyz="0 0 0" rpy="0 0 0" />
+      <geometry>
+          <mesh filename="file:///home/nizan/catkin_ws/src/face_scanner_ros/face_database/bust/bust_collision3.stl"/>
+      </geometry>
+      </collision>
+    </link> -->
+    <!-- <joint name="face_joint" type="fixed">
     <parent link="${prefix}base_link"/>
     <child link="face_link"/>
     <origin rpy="${pi / 2} 0 ${pi}" xyz="${face_x} ${face_y} ${face_z}"/>
-    </joint>
+    </joint> -->
+    <!-- <joint name="bust_joint" type="fixed">
+        <parent link="face_link"/>
+        <child link="bust_link"/>
+        <origin rpy="0 0 0" xyz="0 0 0"/>
+    </joint> -->
     <joint name="${prefix}table-base_link" type="fixed">
       <origin xyz="0 0 ${table_height}" rpy="0 0 0"/>

Commit message: adding end effector

File: ur_description/urdf/inc/ur_macro.xacro (robot description, xacro)
@@ -318,23 +318,5 @@
         <origin xyz="0 0 0" rpy="0 0 0" />
         <geometry>
-          <mesh filename="package://gemmapp_ros/meshes/ee/temptu_airpod_airbrush.stl"/>
-        </geometry>
-        <material name="temptu_airpod_airbrush">
-          <color rgba="1 ${186.0/255.0} ${172.0/255.0} 1" />
-        </material>
-      </visual>
-      <visual>
-        <origin xyz="0 0 0" rpy="0 0 0" />
-        <geometry>
-          <mesh filename="package://gemmapp_ros/meshes/ee/temptu_airpod_camera.stl"/>
-        </geometry>
-        <material name="temptu_airpod_camera">
-          <color rgba="${20.0/255.0} ${20.0/255.0} ${240.0/255.0} 1" />
-        </material>
-      </visual>
-      <visual>
-        <origin xyz="0 0 0" rpy="0 0 0" />
-        <geometry>
-          <mesh filename="package://gemmapp_ros/meshes/ee/temptu_airpod_gripper.stl"/>
+          <mesh filename="package://gemmapp_ros/meshes/ee/HAX_maRC_V1/gripper.stl"/>
         </geometry>
         <material name="temptu_airpod_gripper">
@@ -345,5 +327,5 @@
         <origin xyz="0 0 0" rpy="0 0 0" />
         <geometry>
-          <mesh filename="package://gemmapp_ros/meshes/ee/temptu_airpod_collision.stl"/>
+          <mesh filename="package://gemmapp_ros/meshes/ee/HAX_maRC_V1/gripper.stl"/>
         </geometry>
       </collision>
@@ -356,5 +338,5 @@
     <link name="${prefix}camera_ee" />
     <joint name="${prefix}tool_temp-camera_ee" type="fixed">
-      <origin xyz="0 -0.038 0.139" rpy="0 0 0"/>
+      <origin xyz="0.04 0.045 0.029" rpy="0 0 0"/>
       <parent link="${prefix}tool_temp"/>
       <child link="${prefix}camera_ee"/>
@@ -363,6 +345,6 @@
     <xacro:property name="calibration_y_angle" value="-0.0290007"/>
     <xacro:property name="x_shift" value="0.0"/>
-    <xacro:property name="y_shift" value="0.017"/>
-    <xacro:property name="z_shift" value="0.15578"/>
+    <xacro:property name="y_shift" value="0.0"/>
+    <xacro:property name="z_shift" value="0.097"/>
     <!-- Start: This setup are meant for 'air-brush' experiments -->
     <link name="${prefix}tool0" />

Commit message: .

File: ur_description/urdf/inc/ur_macro.xacro (robot description, xacro)
@@ -338,5 +338,5 @@
     <link name="${prefix}camera_ee" />
     <joint name="${prefix}tool_temp-camera_ee" type="fixed">
-      <origin xyz="0.04 0.045 0.029" rpy="0 0 0"/>
+      <origin xyz="-0.014831710090098777 0.04333403233743426 0.03746148313645714" rpy="0 0 0"/>
       <parent link="${prefix}tool_temp"/>
       <child link="${prefix}camera_ee"/>

Commit message: .

File: ur_description/urdf/inc/ur_macro.xacro (robot description, xacro)
@@ -342,6 +342,6 @@
       <child link="${prefix}camera_ee"/>
     </joint>
-    <xacro:property name="calibration_x_angle" value="-0.0572047"/>
-    <xacro:property name="calibration_y_angle" value="-0.0290007"/>
+    <xacro:property name="calibration_x_angle" value="-0.0230358"/>
+    <xacro:property name="calibration_y_angle" value="-0.0370216"/>
     <xacro:property name="x_shift" value="0.0"/>
     <xacro:property name="y_shift" value="0.0"/>

Commit message: .

File: ur_description/urdf/inc/ur_macro.xacro (robot description, xacro)
@@ -342,8 +342,8 @@
       <child link="${prefix}camera_ee"/>
     </joint>
-    <xacro:property name="calibration_x_angle" value="-0.0230358"/>
-    <xacro:property name="calibration_y_angle" value="-0.0370216"/>
-    <xacro:property name="x_shift" value="0.0"/>
-    <xacro:property name="y_shift" value="0.0"/>
+    <xacro:property name="calibration_x_angle" value="0.03312809"/>
+    <xacro:property name="calibration_y_angle" value="0.035356865"/>
+    <xacro:property name="x_shift" value="-0.00403778"/>
+    <xacro:property name="y_shift" value="-0.00062246"/>
     <xacro:property name="z_shift" value="0.097"/>
     <!-- Start: This setup are meant for 'air-brush' experiments -->

Commit message: .

File: ur_description/urdf/inc/ur_macro.xacro (robot description, xacro)
@@ -318,5 +318,5 @@
         <origin xyz="0 0 0" rpy="0 0 0" />
         <geometry>
-          <mesh filename="package://gemmapp_ros/meshes/ee/HAX_maRC_V1/gripper.stl"/>
+          <mesh filename="package://gemmapp_ros/meshes/ee/HAX_Nick_V1/ee.stl"/>
         </geometry>
         <material name="temptu_airpod_gripper">
@@ -327,5 +327,5 @@
         <origin xyz="0 0 0" rpy="0 0 0" />
         <geometry>
-          <mesh filename="package://gemmapp_ros/meshes/ee/HAX_maRC_V1/gripper.stl"/>
+          <mesh filename="package://gemmapp_ros/meshes/ee/HAX_Nick_V1/ee.stl"/>
         </geometry>
       </collision>
@@ -338,13 +338,13 @@
     <link name="${prefix}camera_ee" />
     <joint name="${prefix}tool_temp-camera_ee" type="fixed">
-      <origin xyz="-0.014831710090098777 0.04333403233743426 0.03746148313645714" rpy="0 0 0"/>
+      <origin xyz="0.006835956674082612 -0.04985659335752479 0.0976500318266122" rpy="0 0 0"/>
       <parent link="${prefix}tool_temp"/>
       <child link="${prefix}camera_ee"/>
     </joint>
-    <xacro:property name="calibration_x_angle" value="0.03312809"/>
-    <xacro:property name="calibration_y_angle" value="0.035356865"/>
-    <xacro:property name="x_shift" value="-0.00403778"/>
-    <xacro:property name="y_shift" value="-0.00062246"/>
-    <xacro:property name="z_shift" value="0.097"/>
+    <xacro:property name="calibration_x_angle" value="0.0"/>
+    <xacro:property name="calibration_y_angle" value="0.0"/>
+    <xacro:property name="x_shift" value="0.0"/>
+    <xacro:property name="y_shift" value="0.0"/>
+    <xacro:property name="z_shift" value="0.1352"/>
     <!-- Start: This setup are meant for 'air-brush' experiments -->
     <link name="${prefix}tool0" />
@@ -355,28 +355,4 @@
     </joint>
     <!-- End: This setup meant for 'air-brush' experiments -->
-    <!-- Start: This setup meant for 'aruco' experiments -->
-    <!-- <link name="${prefix}tool0">
-      <visual>
-        <origin xyz="0 0 -0.015" rpy="0 0 0" />
-        <geometry>
-          <box size="0.2 0.2 0.03" />
-        </geometry>
-        <material name="green">
-          <color rgba="0 1 0 1" />
-        </material>
-      </visual>
-      <collision>
-        <origin xyz="0 0 -0.015" rpy="0 0 0" />
-        <geometry>
-          <box size="0.2 0.2 0.03" />
-        </geometry>
-      </collision>
-    </link>
-    <joint name="${prefix}flange-tool0" type="fixed">
-      <origin xyz="0.014 0 0" rpy="${pi/2.0} 0 ${pi/2.0}"/>
-      <parent link="${prefix}flange"/>
-      <child link="${prefix}tool0"/>
-    </joint> -->
-    <!-- End: This setup meant for 'aruco' experiments -->
     <xacro:property name="table_height" value="0.77"/>
     <xacro:property name="face_x" value="0"/>

Commit message: adding laser

File: ur_description/urdf/inc/ur_macro.xacro (robot description, xacro)
@@ -355,4 +355,10 @@
     </joint>
     <!-- End: This setup meant for 'air-brush' experiments -->
+    <link name="${prefix}laser_ee" />
+    <joint name="${prefix}tool_temp-laser_ee" type="fixed">
+      <origin xyz="0 0.014 0" rpy="0 0 0"/>
+      <parent link="${prefix}tool0"/>
+      <child link="${prefix}laser_ee"/>
+    </joint>
     <xacro:property name="table_height" value="0.77"/>
     <xacro:property name="face_x" value="0"/>

Commit message: rename

File: ur_description/urdf/inc/ur_macro.xacro (robot description, xacro)
@@ -318,5 +318,5 @@
         <origin xyz="0 0 0" rpy="0 0 0" />
         <geometry>
-          <mesh filename="package://gemmapp_ros/meshes/ee/HAX_Nick_V1/ee.stl"/>
+          <mesh filename="package://gemma_makeup/meshes/ee/HAX_Nick_V1/ee.stl"/>
         </geometry>
         <material name="temptu_airpod_gripper">
@@ -327,5 +327,5 @@
         <origin xyz="0 0 0" rpy="0 0 0" />
         <geometry>
-          <mesh filename="package://gemmapp_ros/meshes/ee/HAX_Nick_V1/ee.stl"/>
+          <mesh filename="package://gemma_makeup/meshes/ee/HAX_Nick_V1/ee.stl"/>
         </geometry>
       </collision>

Commit message: .

File: ur_description/urdf/inc/ur_macro.xacro (robot description, xacro)
@@ -379,53 +379,4 @@
       </collision>
     </link>
-    <!-- <link name="face_link">
-        <visual>
-        <origin xyz="0 0 0" rpy="0 0 0" />
-        <geometry>
-          <mesh filename="file:///home/nizan/catkin_ws/src/face_scanner_ros/face_database/eliane/eliane_aligned.dae"/>
-        </geometry>
-      </visual>
-      <collision>
-        <origin xyz="0 0 0" rpy="0 0 0" />
-        <geometry>
-          <mesh filename="file:///home/nizan/catkin_ws/src/face_scanner_ros/face_database/eliane/eliane_aligned_collision.dae"/>
-        </geometry>
-      </collision>
-      <inertial>
-            <origin rpy="0 0 0" xyz="0.043 0.001 0.002" />
-            <mass value="0.1" />
-            <inertia ixx="0.000348958333333" ixy="0" ixz="0" iyy="0.000348958333333" iyz="0" izz="3.125e-05" />
-        </inertial>
-    </link> -->
-    <!-- <link name="bust_link">
-      <collision>
-      <origin xyz="0 0 0" rpy="0 0 0" />
-      <geometry>
-          <mesh filename="file:///home/nizan/catkin_ws/src/face_scanner_ros/face_database/bust/bust_collision1.stl"/>
-      </geometry>
-      </collision>
-      <collision>
-      <origin xyz="0 0 0" rpy="0 0 0" />
-      <geometry>
-          <mesh filename="file:///home/nizan/catkin_ws/src/face_scanner_ros/face_database/bust/bust_collision2.stl"/>
-      </geometry>
-      </collision>
-      <collision>
-      <origin xyz="0 0 0" rpy="0 0 0" />
-      <geometry>
-          <mesh filename="file:///home/nizan/catkin_ws/src/face_scanner_ros/face_database/bust/bust_collision3.stl"/>
-      </geometry>
-      </collision>
-    </link> -->
-    <!-- <joint name="face_joint" type="fixed">
-    <parent link="${prefix}base_link"/>
-    <child link="face_link"/>
-    <origin rpy="${pi / 2} 0 ${pi}" xyz="${face_x} ${face_y} ${face_z}"/>
-    </joint> -->
-    <!-- <joint name="bust_joint" type="fixed">
-        <parent link="face_link"/>
-        <child link="bust_link"/>
-        <origin rpy="0 0 0" xyz="0 0 0"/>
-    </joint> -->
     <joint name="${prefix}table-base_link" type="fixed">
       <origin xyz="0 0 ${table_height}" rpy="0 0 0"/>

Commit message: .

File: ur_description/urdf/inc/ur_macro.xacro (robot description, xacro)
@@ -342,21 +342,36 @@
       <child link="${prefix}camera_ee"/>
     </joint>
-    <xacro:property name="calibration_x_angle" value="0.0"/>
-    <xacro:property name="calibration_y_angle" value="0.0"/>
-    <xacro:property name="x_shift" value="0.0"/>
-    <xacro:property name="y_shift" value="0.0"/>
-    <xacro:property name="z_shift" value="0.1352"/>
-    <!-- Start: This setup are meant for 'air-brush' experiments -->
+    <xacro:property name="airbrush_calib_x_angle" value="0.0"/>
+    <xacro:property name="airbrush_calib_y_angle" value="0.0"/>
+    <xacro:property name="airbrush_calib_x_shift" value="0.0"/>
+    <xacro:property name="airbrush_calib_y_shift" value="0.0"/>
+    <xacro:property name="airbrush_calib_z_shift" value="0.0"/>
+    <link name="${prefix}tool0_no_calib" />
+    <joint name="${prefix}tool_temp-tool0_no_calib" type="fixed">
+      <origin xyz="0 0 0.1352" rpy="0 0 0"/>
+      <parent link="${prefix}tool_temp"/>
+      <child link="${prefix}tool0_no_calib"/>
+    </joint>
     <link name="${prefix}tool0" />
-    <joint name="${prefix}tool_temp-tool0" type="fixed">
-      <origin xyz="${x_shift} ${y_shift} ${z_shift}" rpy="${calibration_y_angle} ${calibration_x_angle} 0"/>
-      <parent link="${prefix}tool_temp"/>
+    <joint name="${prefix}tool0_no_calib-tool0" type="fixed">
+      <origin xyz="${airbrush_calib_x_shift} ${airbrush_calib_y_shift} ${airbrush_calib_z_shift}" rpy="${airbrush_calib_y_angle} ${airbrush_calib_x_angle} 0"/>
+      <parent link="${prefix}tool0_no_calib"/>
       <child link="${prefix}tool0"/>
     </joint>
-    <!-- End: This setup meant for 'air-brush' experiments -->
+    <link name="${prefix}laser_no_calib_ee" />
+    <joint name="${prefix}tool0_no_calib-laser_no_calib_ee" type="fixed">
+      <origin xyz="0 0.014 0" rpy="0 0 0"/>
+      <parent link="${prefix}tool0_no_calib"/>
+      <child link="${prefix}laser_no_calib_ee"/>
+    </joint>
+    <xacro:property name="laser_calib_x_angle" value="0.0"/>
+    <xacro:property name="laser_calib_y_angle" value="0.0"/>
+    <xacro:property name="laser_calib_x_shift" value="0.0"/>
+    <xacro:property name="laser_calib_y_shift" value="0.0"/>
+    <xacro:property name="laser_calib_z_shift" value="0.0"/>
     <link name="${prefix}laser_ee" />
-    <joint name="${prefix}tool_temp-laser_ee" type="fixed">
-      <origin xyz="0 0.014 0" rpy="0 0 0"/>
-      <parent link="${prefix}tool0"/>
+    <joint name="${prefix}laser_no_calib_ee-laser_ee" type="fixed">
+      <origin xyz="${laser_calib_x_shift} ${laser_calib_y_shift} ${laser_calib_z_shift}" rpy="${laser_calib_y_angle} ${laser_calib_x_angle} 0"/>
+      <parent link="${prefix}laser_no_calib_ee"/>
       <child link="${prefix}laser_ee"/>
     </joint>

Commit message: .

File: ur_description/urdf/inc/ur_macro.xacro (robot description, xacro)
@@ -384,5 +384,5 @@
         <origin xyz="0 0 ${table_height}" rpy="0 0 0" />
         <geometry>
-          <mesh filename="file:///home/nizan/catkin_ws/src/gemmaD_robot_ros/gemmad_robot_description/stl/table/full_table.dae"/>
+          <mesh filename="$(find gemma_face_scanner)/face_database/table/full_table.dae"/>
         </geometry>
       </visual>
@@ -390,5 +390,5 @@
         <origin xyz="0 0 ${table_height}" rpy="0 0 0" />
         <geometry>
-          <mesh filename="file:///home/nizan/catkin_ws/src/gemmaD_robot_ros/gemmad_robot_description/stl/table/full_table.dae"/>
+          <mesh filename="$(find gemma_face_scanner)/face_database/table/full_table.dae"/>
         </geometry>
       </collision>

Commit message: .

File: ur_description/urdf/inc/ur_macro.xacro (robot description, xacro)
@@ -384,5 +384,5 @@
         <origin xyz="0 0 ${table_height}" rpy="0 0 0" />
         <geometry>
-          <mesh filename="$(find gemma_face_scanner)/face_database/table/full_table.dae"/>
+          <mesh filename="package://gemma_face_scanner/face_database/table/full_table.dae"/>
         </geometry>
       </visual>
@@ -390,5 +390,5 @@
         <origin xyz="0 0 ${table_height}" rpy="0 0 0" />
         <geometry>
-          <mesh filename="$(find gemma_face_scanner)/face_database/table/full_table.dae"/>
+          <mesh filename="package://gemma_face_scanner/face_database/table/full_table.dae"/>
         </geometry>
       </collision>
